File: Synthesizer_HW.kicad_pcb (KiCad board)
At the start: 2 copper layers, 142.5 x 77.2 mm, 116 parts, among them J1 +5V_DC, J1&1 Selector, J2 USB_B_Micro, J3 EXT_REF_IN, J4 RF OUT1, J5 RF OUT2, Q1 BC857, Q2 BC847, Q3 BC847, Q4 IRLML5203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

Commit message: board WIP, now editing silkscreen
Parts:
- removed C13: 100n, Capacitor_SMD:C_0603_1608Metric
- removed H1, H2, H3, H4: MountingHole_Pad, MountingHole:MountingHole_3.2mm_M3_Pad_Via
- added D5: Status1, LED_SMD:LED_0603_1608Metric, F.Cu at (140.5, 51.9)
- added D6: Status2, LED_SMD:LED_0603_1608Metric, F.Cu at (142.0, 51.9)
- added FB5: BLM18PG471, Inductor_SMD:L_0603_1608Metric, F.Cu at (117.1, 63.7)
- added FB6: BLM18PG471, Inductor_SMD:L_0603_1608Metric, F.Cu at (117.2, 72.6)
- added FB7: BLM18PG471, Inductor_SMD:L_0603_1608Metric, F.Cu at (126.3, 60.6)
- added R30: 0R, Resistor_SMD:R_0603_1608Metric, F.Cu at (115.7, 63.7)
- added R31: 0R, Resistor_SMD:R_1206_3216Metric, F.Cu at (121.0, 57.7)
- added R32: 0R, Resistor_SMD:R_1206_3216Metric_Pad1.42x1.75mm_HandSolder, F.Cu at (134.8, 66.6)
- added R33: 0R, Resistor_SMD:R_1206_3216Metric_Pad1.42x1.75mm_HandSolder, F.Cu at (132.6, 66.6)
- added R34: 1k, Resistor_SMD:R_0603_1608Metric, F.Cu at (139.1, 53.6)
- added R35: 1k, Resistor_SMD:R_0603_1608Metric, F.Cu at (142.0, 55.4)
- C49: footprint Capacitor_SMD:C_0603_1608Metric -> Capacitor_SMD:C_0805_2012Metric
- D3, D4: footprint LED_SMD:LED_0805_2012Metric -> LED_SMD:LED_0603_1608Metric
- J1&1: footprint Connector_PinHeader_1.00mm:PinHeader_2x02_P1.00mm_Horizontal -> Connector_PinHeader_2.54mm:PinHeader_2x02_P2.54mm_Horizontal
- R14, R23, R27, R28, R9: footprint Resistor_SMD:R_0603_1608Metric -> Resistor_SMD:R_0805_2012Metric
- X1: footprint Crystal:Crystal_SMD_Abracon_ABM8G-4Pin_3.2x2.5mm -> KLALIB_Crystal:Crystal_SMD_4Pin_3.2x2.5mm
- moved J3 57.4 mm to (153.8, 78.3), turned to 180 degrees
- moved J4 19.6 mm to (103.8, 56.6)
- moved J1&1 10.2 mm to (145.2, 64.9)
- moved C42 10.1 mm to (111.6, 75.7)
- moved J5 9.61 mm to (103.8, 72.6)
- moved C44 9.40 mm to (111.6, 77.2), turned to 0 degrees
- moved C38 9.16 mm to (117.3, 79.1)
- moved Q4 9.16 mm to (114.8, 79.1)
- moved R24 9.16 mm to (118.7, 79.1)
- moved FB3 8.58 mm to (118.7, 73.8), turned to 90 degrees
- moved R1 7.35 mm to (133.6, 73.2), turned to 180 degrees
- moved U6 7.33 mm to (112.2, 72.3)
- moved C47 6.84 mm to (111.6, 78.6), turned to 0 degrees
- moved R5 6.68 mm to (141.2, 79.8)
- moved R23 6.67 mm to (148.1, 74.3)
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Connections:
- C10 pad 2: VDDA -> Net-(C10-Pad2)
- C12 pad 1: VDDA -> Net-(C10-Pad2)
- C14 pad 2: VDDA -> Net-(C14-Pad2)
- C16 pad 1: VDDA -> Net-(C14-Pad2)
- C26 pad 1: VDD -> /VDD1
- C27 pad 2: VDD -> /VDD1
- C30 pad 2: VDDA -> Net-(C30-Pad2)
- C31 pad 1: VDDA -> Net-(C30-Pad2)
- C33 pad 2: VDDA -> Net-(C30-Pad2)
- C34 pad 1: VDDA -> Net-(C30-Pad2)
- D4 pad 2: +5V -> Net-(D4-Pad2)
- FB2 pad 1: VDDA -> Net-(FB2-Pad1)
- FB3 pad 1: VDDA -> Net-(FB2-Pad1)
- J1 pad 1: GND -> Net-(FB1-Pad2)
- J1 pad 2: Net-(FB1-Pad2) -> GND
- Q3 pad 3: Net-(Q3-Pad3) -> Net-(D4-Pad1)
- R15 pad 1: VDDA -> Net-(C30-Pad2)
- R16 pad 2: Net-(C28-Pad1) -> Net-(R16-Pad2)
- R17 pad 1: VDDA -> Net-(C30-Pad2)
- R21 pad 1: VDDA -> Net-(C30-Pad2)
- R22 pad 1: VDDA -> Net-(C30-Pad2)
- R23 pad 1: Net-(D4-Pad1) -> +5V
- R23 pad 2: Net-(Q3-Pad3) -> Net-(D4-Pad2)
- R6 pad 2: VDD -> /VDD1
- U3 pad 10: /INT_REF -> Net-(R32-Pad2)
- U3 pad 19: (no net) -> Net-(R35-Pad1)
- U3 pad 20: (no net) -> Net-(R34-Pad1)
- U4 pad 10: VDDA -> Net-(C10-Pad2)
- U4 pad 28: VDD -> /VDD1
- U4 pad 6: VDDA -> Net-(C14-Pad2)
Routing:
- net +5V: track 0.00 -> 99.1 mm
- net GND: track 0.00 -> 52.6 mm, vias 0 -> 393
- net VDD: track 0.00 -> 30.6 mm
- net Net-(C38-Pad2): track 0.00 -> 30.6 mm
- net Net-(C5-Pad1): track 0.00 -> 26.4 mm
- net Net-(C40-Pad2): track 0.00 -> 23.1 mm
- net Net-(C10-Pad2): track 0.00 -> 21.9 mm
- net Net-(C25-Pad1): track 0.00 -> 19.9 mm
- net VDDA: track 0.00 -> 18.2 mm
- net Net-(C28-Pad1): track 0.00 -> 18.0 mm
- net Net-(C2-Pad2): track 0.00 -> 17.2 mm
- net Net-(JP1-Pad1): track 0.00 -> 17.1 mm
- net /DOUBLER_EN: track 0.00 -> 14.8 mm
- net Net-(C18-Pad2): track 0.00 -> 14.2 mm
- net Net-(D3-Pad1): track 0.00 -> 13.7 mm
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- added copper zone on B.Cu, net GND
- added copper zone on F.Cu, net GND
- added copper zone on F.Cu, net Net-(C30-Pad2)
- added copper zone on F.Cu, net Net-(C48-Pad1)
- added copper zone on F.Cu, net Net-(C48-Pad2)
- added copper zone on F.Cu, net Net-(J5-Pad1)
Other:
- board size 142.5 x 77.2 mm -> 59.5 x 39 mm
- net class Default: trace_width 0.25 -> 0.254; via_dia 0.8 -> 0.6; via_drill 0.4 -> 0.3
- rule trace_min: 0.1524 -> 0
- rule via_min_size: 0.4 -> 0.6

Commit message: first almost done version, with debug interface,
Parts:
- removed D5: Status1, LED_SMD:LED_0603_1608Metric
- removed D6: Status2, LED_SMD:LED_0603_1608Metric
- removed R34, R35: 1k, Resistor_SMD:R_0603_1608Metric
- added D7: OUT2_Active, LED_SMD:LED_0603_1608Metric, F.Cu at (117.5, 81.1)
- added D8: OUT1_Active, LED_SMD:LED_0603_1608Metric, F.Cu at (109.3, 48.8)
- added J6: SWD, Connector_Molex:Molex_PicoBlade_53047-0410_1x04_P1.25mm_Vertical, F.Cu at (141.7, 52.4)
- added R36: 1k, Resistor_SMD:R_0603_1608Metric, F.Cu at (114.5, 81.1)
- added R37: 1k, Resistor_SMD:R_0603_1608Metric, F.Cu at (111.7, 49.4)
- added TP1: PLO_LE, TestPoint:TestPoint_Pad_D1.0mm, F.Cu at (128.2, 58.6)
- added TP2: PLO_DATA, TestPoint:TestPoint_Pad_D1.0mm, F.Cu at (128.9, 60.8)
- added TP3: PLO_CLK, TestPoint:TestPoint_Pad_D1.0mm, F.Cu at (128.0, 64.2)
- added TP7: GND, TestPoint:TestPoint_Loop_D1.80mm_Drill1.0mm_Beaded, F.Cu at (128.5, 54.4)
- moved R7 1.08 mm to (129.3, 56.8)
- moved C38 0.52 mm to (117.2, 78.5)
- moved Q4 0.52 mm to (114.7, 78.5)
- moved R24 0.52 mm to (118.6, 78.5)
- moved R11 0.21 mm to (130.7, 59.4)
- moved R12 0.18 mm to (130.7, 60.8)
- moved R13 0.16 mm to (130.6, 62.3)
- moved C43 0.14 mm to (109.3, 51.8)
- moved C46 0.14 mm to (110.8, 51.8)
- moved C44 0.09 mm to (111.5, 77.2)
- moved C42 0.09 mm to (111.5, 75.7)
- moved C47 0.09 mm to (111.5, 78.6)
- moved C50 0.09 mm to (111.5, 80.1)
Connections:
- net Net-(C15-Pad2) renamed /~RST
- U3 pad 19: Net-(R35-Pad1) -> /SWDIO
- U3 pad 20: Net-(R34-Pad1) -> /SWCLK
Routing:
- net /~RST: track 5.67 -> 11.0 mm, vias 0 -> 1
- net Net-(R35-Pad1): track 2.91 -> 0.00 mm
- net /SWCLK: track 0.00 -> 2.76 mm
- net /SWDIO: track 0.00 -> 2.51 mm
- net Net-(R7-Pad1): track 7.96 -> 10.1 mm
- net Net-(D6-Pad2): track 1.92 -> 0.00 mm
- net /PLO_LE: track 6.95 -> 8.61 mm
- net Net-(C42-Pad2): track 7.98 -> 9.63 mm
- net Net-(D8-Pad2): track 0.00 -> 1.60 mm
- net Net-(C43-Pad2): track 4.91 -> 6.44 mm
- net Net-(D5-Pad2): track 1.52 -> 0.00 mm
- net GND: track 52.6 -> 54.1 mm, vias 393 -> 391
- net Net-(D7-Pad2): track 0.00 -> 1.44 mm
- net Net-(R34-Pad1): track 1.41 -> 0.00 mm
- net /PLO_DATA: track 5.69 -> 6.21 mm
Other:
- board text added: "23,5 MHz 6 GHz"
- board text added: "5 GHz 12 GHz"
- board text added: "CLK"
- board text added: "DATA"
- board text added: "DC+5V"
- board text added: "EXT REF"
- board text added: "F-L"
- board text added: "GND"
- board text added: "LE"
- board text added: "LOCK"
- board text added: "OUT1"
- board text added: "OUT1_Active"
- board text added: "OUT2"
- board text added: "OUT2_Active"
- board text added: "REF"
- board text added: "SWCLK"
- board text added: "SWD"
- board text added: "SWDIO"
- board text added: "~CLK"

Commit message: latest vers., after correc., added moun. holes
Parts:
- added H1: MountingHole_Pad, MountingHole:MountingHole_3.2mm_M3_Pad_Via, F.Cu at (102.8, 47.0)
- added H2: MountingHole_Pad, MountingHole:MountingHole_3.2mm_M3_Pad_Via, F.Cu at (147.8, 47.0)
- added H3: MountingHole_Pad, MountingHole:MountingHole_3.2mm_M3_Pad_Via, F.Cu at (147.8, 81.5)
- added H4: MountingHole_Pad, MountingHole:MountingHole_3.2mm_M3_Pad_Via, F.Cu at (102.8, 81.8)
- J2: value USB_B_Micro -> USB_B_Mini; footprint Connector_USB:USB_Micro-B_Molex_47346-0001 -> Connector_USB:USB_Mini-B_Lumberg_2486_01_Horizontal
- J6: moved to B.Cu
- moved D2 5.24 mm to (146.2, 54.4), turned to -90 degrees
- moved FB1 4.31 mm to (153.0, 52.5), turned to 0 degrees
- moved C4 4.21 mm to (148.5, 57.7), turned to 180 degrees
- moved J7 2.85 mm to (146.5, 67.5)
- moved D3 2.39 mm to (147.1, 76.7), turned to 0 degrees
- moved J1 2.24 mm to (153.1, 48.8)
- moved D1 2.20 mm to (149.7, 53.7)
- moved U1 2.09 mm to (149.0, 60.3)
- moved D4 1.96 mm to (147.1, 72.6), turned to 0 degrees
- moved C6 1.91 mm to (144.0, 51.3)
- moved F1 1.85 mm to (149.7, 51.2)
- moved FB4 1.58 mm to (150.8, 56.9)
- moved R23 1.52 mm to (149.6, 74.3)
- moved J2 1.38 mm to (155.7, 59.7)
- moved J3 1.23 mm to (155.0, 78.3)
- renumbered J1&1 to J7
Routing:
- net GND: track 54.1 -> 63.3 mm, vias 391 -> 380
- net Net-(D3-Pad1): track 13.7 -> 9.10 mm
- net Net-(J1&1-Pad4): track 13.5 -> 16.8 mm
- net Net-(J1&1-Pad2): track 11.7 -> 14.6 mm
- net Net-(C6-Pad1): track 7.55 -> 5.02 mm
- net Net-(F1-Pad2): track 1.47 -> 2.64 mm
- net /USB_D+: track 10.4 -> 9.54 mm
- net Net-(C2-Pad2): track 17.2 -> 17.9 mm
- net Net-(D1-Pad1): track 2.07 -> 1.54 mm
Other:
- board size 59.5 x 39 mm -> 61 x 42.2 mm
- board text added: "~RST"
- board text removed: "23,5 MHz 6 GHz"
- board text removed: "5 GHz 12 GHz"
- board text removed: "~CLK"

Commit message: last version-send to prof. with dimensions
Parts:
- removed D7: OUT2_Active, LED_SMD:LED_0603_1608Metric
- added D5: LG L29K-F2J1-24, LED_SMD:LED_0603_1608Metric, F.Cu at (117.5, 81.0)
- C29, C48: value 22p -> 100p
- C42: value 2p -> 2p2
- C43, C44: value 22p -> 10p
- D3: value EXT_REF_ACTIVE -> LG L29K-F2J1-24
- D4: value Lock/Test -> LG L29K-F2J1-24
- D8: value OUT1_Active -> LG L29K-F2J1-24
- F1: value Fuse -> ERBRE0R50V
- R32, R33: footprint Resistor_SMD:R_1206_3216Metric_Pad1.42x1.75mm_HandSolder -> Resistor_SMD:R_1206_3216Metric
- U1: footprint Package_TO_SOT_SMD:SOT-23-6 -> Package_TO_SOT_SMD:SOT-666
- moved F1 0.76 mm to (149.7, 51.9)
- moved D1 0.75 mm to (149.7, 54.4)
- moved FB4 0.72 mm to (150.8, 57.7)
- moved C4 0.70 mm to (148.5, 58.4)
- moved D2 0.57 mm to (146.8, 54.4)
- moved H3 0.56 mm to (148.0, 82.0)
- moved H4 0.35 mm to (103.0, 82.0)
- moved H1 0.25 mm to (103.0, 47.0)
- moved H2 0.25 mm to (148.0, 47.0)
- moved D3 0.19 mm to (147.1, 76.5)
- moved C9 0.19 mm to (133.8, 63.4)
- moved R9 0.19 mm to (137.2, 63.4)
- moved J1 0.19 mm to (153.3, 48.8)
- moved J3 0.16 mm to (155.2, 78.3)
- moved C6 0.07 mm to (144.0, 51.2)
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Routing:
- net GND: track 63.3 -> 65.0 mm, vias 380 -> 386
- net /USB_D+: track 9.54 -> 10.7 mm
- net /PLO_MUXOUT: track 10.4 -> 9.65 mm
- net VBUS: track 11.5 -> 10.8 mm
- net Net-(F1-Pad2): track 2.64 -> 1.99 mm
Other:
- board size 61 x 42.2 mm -> 61 x 43 mm

Commit message: version v0.1 for fabrication
Parts:
- U7: footprint Package_DFN_QFN:DFN-10-1EP_3x3mm_P0.5mm_EP1.65x2.38mm_ThermalVias -> KLALIB_Housing:DFN-10-1EP_3x3mm_P0.5mm_EP1.65x2.38mm_ThermalVias
- moved J7 0.93 mm to (147.4, 67.5)
- moved J3 0.51 mm to (155.7, 78.3)
- moved J1 0.51 mm to (153.8, 48.8)
- moved H2 0.50 mm to (148.5, 47.0)
- moved H3 0.50 mm to (148.5, 82.0)
- moved J2 0.10 mm to (155.8, 59.7)
Routing:
- net GND: track 65.0 -> 66.6 mm, vias 386 -> 398
- net Net-(J7-Pad4): track 16.8 -> 17.5 mm
- net Net-(J7-Pad2): track 14.6 -> 15.1 mm
Other:
- board size 61 x 43 mm -> 61.5 x 43 mm
- board text added: "Synthesizer v0.1 FKU 12/2019"
